Commit message: modified:   rplidar_ros/launch/rplidar_a2m8_launch.py

File: hoist_base/urdf/hoist.urdf (robot description, URDF)
Before this commit: robot robot, 9 links, 8 joints
Joints:
- removed joint hokuyo_joint
- added joint laser_joint: type fixed, parent base_link, child laser_frame, origin xyz=0.0 0.0 -0.0501 rpy=3.141592 0 0, axis 0 1 0

Commit message: modified:   hoist_base/config/ekf_gazebo.yaml 	modified:   hoist_base/urdf/hoist.urdf

File: hoist_base/urdf/hoist.urdf (robot description, URDF)
Before this commit: robot robot, 9 links, 8 joints
Links:
- removed link dummy
- link base_footprint: geometry visual box size=0.425 0.4596 0.001
Joints:
- removed joint dummy_joint

Commit message: modified:   hoist_base/urdf/hoist.urdf

File: hoist_base/urdf/hoist.urdf (robot description, URDF)
Before this commit: robot robot, 8 links, 7 joints
Joints:
- joint laser_joint: origin xyz=0.0 0.0 -0.0501 rpy=3.141592 0 0 -> xyz=0.0 0.0 -0.0051 rpy=3.141592 0 3.141592

Commit message: changes imu yaw

File: hoist_base/urdf/hoist.urdf (robot description, URDF)
Before this commit: robot robot, 8 links, 7 joints
Joints:
- joint imu_joint: origin xyz=0.092 0 -0.035 rpy=0 0 0 -> xyz=0.092 0 -0.035 rpy=0 0 3.14159

Commit message: modified:   hoist_base/urdf/hoist.urdf

File: hoist_base/urdf/hoist.urdf (robot description, URDF)
Before this commit: robot robot, 8 links, 7 joints
Joints:
- joint imu_joint: origin xyz=0.092 0 -0.035 rpy=0 0 3.14159 -> xyz=0.092 0 -0.035 rpy=3.14159 0 0

Commit message: modified:   hoist_base/urdf/hoist.urdf

File: hoist_base/urdf/hoist.urdf (robot description, URDF)
Before this commit: robot robot, 8 links, 7 joints
Joints:
- joint imu_joint: origin xyz=0.092 0 -0.035 rpy=3.14159 0 0 -> xyz=0.092 0 -0.035 rpy=0 0 0

Commit message: modified:   hoist_base/config/ekf.yaml

File: hoist_base/urdf/hoist.urdf (robot description, URDF)
Before this commit: robot robot, 8 links, 7 joints
Joints:
- joint imu_joint: origin xyz=0.092 0 -0.035 rpy=0 0 3.14159 -> xyz=0.092 0 -0.035 rpy=3.14159 0.0 0.0
